Commit message: updated iiwa02 with correct file path

File: resources/05-unity-kuka/kuka_iiwa02.urdf (robot description, URDF)
Before this commit: robot kuka_iiwa, 8 links, 7 joints
Links:
- link base_link: geometry visual mesh filename=meshes/base.obj scale=1 1 1
- link link0: geometry visual mesh filename=meshes/link0.obj scale=1 1 1
- link link1: geometry visual mesh filename=meshes/link1.obj scale=1 1 1
- link link2: geometry visual mesh filename=meshes/link2.obj scale=1 1 1
- link link3: geometry visual mesh filename=meshes/link3.obj scale=1 1 1
- link link4: geometry visual mesh filename=meshes/link4.obj scale=1 1 1
- link link5: geometry visual mesh filename=meshes/link5.obj scale=1 1 1
- link link6: geometry collision mesh filename=meshes/link6.obj scale=1 1 1; visual mesh filename=meshes/link6.obj scale=1 1 1
